Commit message: Add files via upload

File: arm/urdf/robot.urdf (robot description, URDF)
Before this commit: robot robot2, 11 links, 10 joints
Links:
- added link camera_link, mass 0.25; collision box size=0.05 0.05 0.05; visual box size=0.05 0.05 0.05
- added link camera_link_optical
Joints:
- added joint camera_joint: type fixed, parent world, child camera_link, origin xyz=0 0 2.2 rpy=0 1.57 0
- added joint camera_optical_joint: type fixed, parent camera_link, child camera_link_optical, origin xyz=0 0 0 rpy=1.57 0 1.57
